Commit message: update model to have contact + gripper, remove old models, update env + example

File: organized_kinova/6dof/urdf/GEN3-LITE.urdf (robot description, URDF)
Before this commit: robot KR7108-URDF, 8 links, 7 joints
Links:
- added link TOOL_FRAME, mass 1e-06
- link ARM: geometry collision mesh filename=../meshes/arm_link.STL; visual mesh filename=../meshes/arm_link.STL
- link BASE: geometry collision mesh filename=../meshes/base_link.STL; visual mesh filename=../meshes/base_link.STL
- link DUMMY: mass None -> 1e-06
- link END_EFFECTOR: mass None -> 1e-06
- link FOREARM: geometry collision mesh filename=../meshes/forearm_link.STL; visual mesh filename=../meshes/forearm_link.STL
- link LOWER_WRIST: geometry collision mesh filename=../meshes/lower_wrist_link.STL; visual mesh filename=../meshes/lower_wrist_link.STL
- link SHOULDER: geometry collision mesh filename=../meshes/shoulder_link.STL; visual mesh filename=../meshes/shoulder_link.STL
- link UPPER_WRIST: geometry collision mesh filename=../meshes/upper_wrist_link.STL; visual mesh filename=../meshes/upper_wrist_link.STL
Joints:
- removed joint END_EFFECTOR
- added joint end_effector_to_dummy: type fixed, parent END_EFFECTOR, child DUMMY, origin xyz=0 0 0 rpy=0 0 0
- added joint tool_frame_joint: type fixed, parent END_EFFECTOR, child TOOL_FRAME, origin xyz=0 0 0.130 rpy=0 0 1.57079632679
- joint J0: limit lower=-2.76 upper=2.76 effort=10 velocity=0.35 -> lower=-2.69 upper=2.69 effort=10 velocity=1.6
- joint J1: limit lower=-2.76 upper=2.76 effort=14 velocity=0.35 -> lower=-2.69 upper=2.69 effort=14 velocity=1.6
- joint J2: limit lower=-2.76 upper=2.76 effort=10 velocity=0.35 -> lower=-2.69 upper=2.69 effort=10 velocity=1.6
- joint J3: limit lower=-2.67 upper=2.67 effort=7 velocity=0.35 -> lower=-2.59 upper=2.59 effort=7 velocity=1.6
- joint J4: limit lower=-2.67 upper=2.67 effort=7 velocity=0.35 -> lower=-2.57 upper=2.57 effort=7 velocity=1.6
- joint J5: limit lower=-2.67 upper=2.67 effort=7 velocity=0.35 -> lower=-2.59 upper=2.59 effort=7 velocity=3.2

File: organized_kinova/6dof/urdf/gen3_lite_macro.xacro (robot description, xacro)
@@ -1,4 +1,6 @@
 <?xml version="1.0"?>
 <robot name="gen3_lite_arm" xmlns:xacro="http://ros.org/wiki/xacro">
+  <!-- Override for offline/MuJoCo: e.g. mesh_prefix_arm="../meshes" with dof=6 and flattened paths in a wrapper xacro. -->
+  <xacro:property name="mesh_prefix_arm" value="package://kortex_description/arms/gen3_lite"/>
   <!-- Propagate last link name information because it is the gripper's parent link -->
   <xacro:property name="last_arm_link" value="dummy_link"/>
@@ -13,14 +15,14 @@
         <origin xyz="0 0 0" rpy="0 0 0" />
         <geometry>
-          <mesh filename="package://kortex_description/arms/gen3_lite/${dof}dof/meshes/base_link.STL" />
-        </geometry>
-        <material name="">
-          <color rgba="0.803 0.824 0.820 1" />
-        </material>
-      </visual>
-      <collision>
-        <origin xyz="0 0 0" rpy="0 0 0" />
-        <geometry>
-          <mesh filename="package://kortex_description/arms/gen3_lite/${dof}dof/meshes/base_link.STL" />
+          <mesh filename="${mesh_prefix_arm}/${dof}dof/meshes/base_link.STL" />
+        </geometry>
+        <material name="">
+          <color rgba="0.803 0.824 0.820 1" />
+        </material>
+      </visual>
+      <collision>
+        <origin xyz="0 0 0" rpy="0 0 0" />
+        <geometry>
+          <mesh filename="${mesh_prefix_arm}/${dof}dof/meshes/base_link.STL" />
         </geometry>
       </collision>
@@ -38,14 +40,14 @@
         <origin xyz="0 0 0" rpy="0 0 0" />
         <geometry>
-          <mesh filename="package://kortex_description/arms/gen3_lite/${dof}dof/meshes/shoulder_link.STL" />
-        </geometry>
-        <material name="">
-          <color rgba="0.803 0.824 0.820 1" />
-        </material>
-      </visual>
-      <collision>
-        <origin xyz="0 0 0" rpy="0 0 0" />
-        <geometry>
-          <mesh filename="package://kortex_description/arms/gen3_lite/${dof}dof/meshes/shoulder_link.STL" />
+          <mesh filename="${mesh_prefix_arm}/${dof}dof/meshes/shoulder_link.STL" />
+        </geometry>
+        <material name="">
+          <color rgba="0.803 0.824 0.820 1" />
+        </material>
+      </visual>
+      <collision>
+        <origin xyz="0 0 0" rpy="0 0 0" />
+        <geometry>
+          <mesh filename="${mesh_prefix_arm}/${dof}dof/meshes/shoulder_link.STL" />
         </geometry>
       </collision>
@@ -59,5 +61,5 @@
       <child link="${prefix}shoulder_link" />
       <axis xyz="0 0 1" />
-      <limit lower="-2.68" upper="2.68" effort="10" velocity="1.6" />
+      <limit lower="-2.69" upper="2.69" effort="10" velocity="1.6" />
     </joint>
     <link name="${prefix}arm_link">
@@ -70,14 +72,14 @@
         <origin xyz="0 0 0" rpy="0 0 0" />
         <geometry>
-          <mesh filename="package://kortex_description/arms/gen3_lite/${dof}dof/meshes/arm_link.STL" />
-        </geometry>
-        <material name="">
-          <color rgba="0.803 0.824 0.820 1" />
-        </material>
-      </visual>
-      <collision>
-        <origin xyz="0 0 0" rpy="0 0 0" />
-        <geometry>
-          <mesh filename="package://kortex_description/arms/gen3_lite/${dof}dof/meshes/arm_link.STL" />
+          <mesh filename="${mesh_prefix_arm}/${dof}dof/meshes/arm_link.STL" />
+        </geometry>
+        <material name="">
+          <color rgba="0.803 0.824 0.820 1" />
+        </material>
+      </visual>
+      <collision>
+        <origin xyz="0 0 0" rpy="0 0 0" />
+        <geometry>
+          <mesh filename="${mesh_prefix_arm}/${dof}dof/meshes/arm_link.STL" />
         </geometry>
       </collision>
@@ -91,5 +93,5 @@
       <child link="${prefix}arm_link" />
       <axis xyz="0 0 1" />
-      <limit lower="-2.61" upper="2.61" effort="14" velocity="1.6" />
+      <limit lower="-2.69" upper="2.69" effort="14" velocity="1.6" />
     </joint>
     <link name="${prefix}forearm_link">
@@ -102,14 +104,14 @@
         <origin xyz="0 0 0" rpy="0 0 0" />
         <geometry>
-          <mesh filename="package://kortex_description/arms/gen3_lite/${dof}dof/meshes/forearm_link.STL" />
-        </geometry>
-        <material name="">
-          <color rgba="0.803 0.824 0.820 1" />
-        </material>
-      </visual>
-      <collision>
-        <origin xyz="0 0 0" rpy="0 0 0" />
-        <geometry>
-          <mesh filename="package://kortex_description/arms/gen3_lite/${dof}dof/meshes/forearm_link.STL" />
+          <mesh filename="${mesh_prefix_arm}/${dof}dof/meshes/forearm_link.STL" />
+        </geometry>
+        <material name="">
+          <color rgba="0.803 0.824 0.820 1" />
+        </material>
+      </visual>
+      <collision>
+        <origin xyz="0 0 0" rpy="0 0 0" />
+        <geometry>
+          <mesh filename="${mesh_prefix_arm}/${dof}dof/meshes/forearm_link.STL" />
         </geometry>
       </collision>
@@ -123,5 +125,5 @@
       <child link="${prefix}forearm_link" />
       <axis xyz="0 0 1" />
-      <limit lower="-2.61" upper="2.61" effort="10" velocity="1.6" />
+      <limit lower="-2.69" upper="2.69" effort="10" velocity="1.6" />
     </joint>
     <link name="${prefix}lower_wrist_link">
@@ -134,14 +136,14 @@
         <origin xyz="0 0 0" rpy="0 0 0" />
         <geometry>
-          <mesh filename="package://kortex_description/arms/gen3_lite/${dof}dof/meshes/lower_wrist_link.STL" />
-        </geometry>
-        <material name="">
-          <color rgba="0.803 0.824 0.820 1" />
-        </material>
-      </visual>
-      <collision>
-        <origin xyz="0 0 0" rpy="0 0 0" />
-        <geometry>
-          <mesh filename="package://kortex_description/arms/gen3_lite/${dof}dof/meshes/lower_wrist_link.STL" />
+          <mesh filename="${mesh_prefix_arm}/${dof}dof/meshes/lower_wrist_link.STL" />
+        </geometry>
+        <material name="">
+          <color rgba="0.803 0.824 0.820 1" />
+        </material>
+      </visual>
+      <collision>
+        <origin xyz="0 0 0" rpy="0 0 0" />
+        <geometry>
+          <mesh filename="${mesh_prefix_arm}/${dof}dof/meshes/lower_wrist_link.STL" />
         </geometry>
       </collision>
@@ -155,5 +157,5 @@
       <child link="${prefix}lower_wrist_link" />
       <axis xyz="0 0 1" />
-      <limit lower="-2.6" upper="2.6" effort="7" velocity="1.6" />
+      <limit lower="-2.59" upper="2.59" effort="7" velocity="1.6" />
     </joint>
     <link name="${prefix}upper_wrist_link">
@@ -166,14 +168,14 @@
         <origin xyz="0 0 0" rpy="0 0 0" />
         <geometry>
-          <mesh filename="package://kortex_description/arms/gen3_lite/${dof}dof/meshes/upper_wrist_link.STL" />
-        </geometry>
-        <material name="">
-          <color rgba="0.803 0.824 0.820 1" />
-        </material>
-      </visual>
-      <collision>
-        <origin xyz="0 0 0" rpy="0 0 0" />
-        <geometry>
-          <mesh filename="package://kortex_description/arms/gen3_lite/${dof}dof/meshes/upper_wrist_link.STL" />
+          <mesh filename="${mesh_prefix_arm}/${dof}dof/meshes/upper_wrist_link.STL" />
+        </geometry>
+        <material name="">
+          <color rgba="0.803 0.824 0.820 1" />
+        </material>
+      </visual>
+      <collision>
+        <origin xyz="0 0 0" rpy="0 0 0" />
+        <geometry>
+          <mesh filename="${mesh_prefix_arm}/${dof}dof/meshes/upper_wrist_link.STL" />
         </geometry>
       </collision>
@@ -187,5 +189,5 @@
       <child link="${prefix}upper_wrist_link" />
       <axis xyz="0 0 1" />
-      <limit lower="-2.53" upper="2.53" effort="7" velocity="1.6" />
+      <limit lower="-2.57" upper="2.57" effort="7" velocity="1.6" />
     </joint>
     <link name="${prefix}end_effector_link"/>
@@ -195,5 +197,5 @@
       <child link="${prefix}end_effector_link" />
       <axis xyz="0 0 1" />
-      <limit lower="-2.6" upper="2.6" effort="7" velocity="3.2" />
+      <limit lower="-2.59" upper="2.59" effort="7" velocity="3.2" />
     </joint>
     <link name="${prefix}dummy_link" />
